File: Hardware/PCB/power.kicad_sch (KiCad schematic)
At the start: 0 parts

Commit message: added buttons
Parts:
- added C10, C12: 22u, symbol Device:C
- added C11, C13: 470n, symbol Device:C
- added C8: 10u, symbol Device:C
- added C9: 100n, symbol Device:C
- added D5: LED, symbol Device:LED
- added L1: 3.9u, symbol Device:L
- added R14: 0R, symbol Device:R
- added R15: 1k2, symbol Device:R
- added TP3: Vbus, symbol Connector:TestPoint
- added TP4: 3.3V, symbol Connector:TestPoint
- added U3: AP63203WU, Package_TO_SOT_SMD:TSOT-23-6, symbol Regulator_Switching:AP63203WU
Connections:
- new net: C11.1, R14.2
- new net: C9.2, L1.1, U3.5 (SW)
- new net: C9.1, U3.6 (BST)
- new net: D5.2 (A), R15.1
- new net +3.3V: C10.1, C12.2, L1.2, R15.2, TP4.1, U3.1 (FB)
- new net GND: C10.2, C11.2, C12.1, C13.2, C8.2, D5.1 (K), U3.4 (GND)
- new net VBUS: C13.1, C8.1, R14.1, TP3.1, U3.2 (EN), U3.3 (IN)
Other:
- note added: "Buck IC 5V->3.3V"
- note added: "PI filter"
- note added: "Power LED"
- note added: "jlc link"
- note added: "voltage testpoints"
